File: RosettaBone_Redux/RBR.kicad_pcb (KiCad board)
At the start: 0 parts

Commit message: Cleanup
Parts:
- added BB101: BeagleBone Black, BeagleBone-Pins, B.Cu at (106.0, 83.8)
- added C301: 100n, CAPC1608x55N, F.Cu at (108.6, 97.2)
- added C302: 100n, CAPC1608x55N, F.Cu at (102.9, 74.9)
- added C501: 100n, CAPC1608x55N, F.Cu at (117.5, 87.6)
- added JP301: HEADER_2X2, pin_strip_2x2, F.Cu at (121.9, 96.5)
- added M101: PCB_GREEN_RMC, OSHW_logo_2, F.Cu at (109.2, 81.3)
- added M102: LOGO_OSHW, PCB_GREEN_RMC, F.Cu at (127.6, 132.1)
- added P101: SOCKET_6_LONG, pin_strip_6, B.Cu at (111.8, 103.5)
- added P8: BB_EXP_CONN, P8P9_PinHeader, B.Cu at (82.5, 61.0)
- added P9: BB_EXP_CONN, P8P9_PinHeader, B.Cu at (82.5, 109.2)
- added R306: 4k7, RESC1608x55N, F.Cu at (108.6, 95.2)
- added R307: 4k7, RESC1608x55N, F.Cu at (108.6, 93.3)
- added R308: 10k, RESC1608x55N, F.Cu at (83.2, 95.2)
- added R309: 10k, RESC1608x55N, F.Cu at (72.4, 66.0)
- added R310: 10k, RESC1608x55N, F.Cu at (92.1, 51.8)
- added R311: 10k, RESC1608x55N, F.Cu at (78.7, 121.4)
- added R312: 10k, RESC1608x55N, F.Cu at (78.7, 116.8)
- added R313: 10k, RESC1608x55N, F.Cu at (78.7, 112.3)
- added R314: 4k7, RESC1608x55N, F.Cu at (142.2, 109.9)
- added R315: 10k, RESC1608x55N, F.Cu at (84.3, 115.8)
- added R316: 10k, RESC1608x55N, F.Cu at (88.4, 115.8)
- added R501: 10k, RESC1608x55N, F.Cu at (236.9, 61.0)
- added R502: 10k, RESC1608x55N, F.Cu at (236.9, 58.4)
- added R503: 10k, RESC1608x55N, F.Cu at (236.9, 55.9)
- added R504: 10k, RESC1608x55N, F.Cu at (236.9, 53.3)
- added R505: 10k, RESC1608x55N, F.Cu at (236.9, 50.8)
- added R506: 10k, RESC1608x55N, F.Cu at (236.9, 48.3)
- added R507: 10k, RESC1608x55N, F.Cu at (236.2, 40.0)
- added R508: 10k, RESC1608x55N, F.Cu at (233.7, 40.0)
- added R509: 10k, RESC1608x55N, F.Cu at (231.1, 40.0)
- added R510: 10k, RESC1608x55N, F.Cu at (228.6, 40.0)
- added SHIELD101: ARDUINO_DUE_SHIELD, ARDUINO_MEGA_DUE_SHIELD_FOOTPRINT_RMC, B.Cu at (55.2, 66.0)
- added U301: 24C256, SOIC127P600X175-8AN, F.Cu at (114.3, 95.2)
- added U302: 74ACT244, SOIC127P1032X265-20N, F.Cu at (181.6, 44.5)
- added U501: 74CBTD3861, SOIC127P1030X265-24N, F.Cu at (204.5, 45.7)
Routing:
- net (no net): track 0.00 -> 4723.8 mm, vias 0 -> 75
- net Z_DIR: track 0.00 -> 42.5 mm
- net Z_STEP: track 0.00 -> 39.3 mm
- net N-00000154: track 0.00 -> 9.84 mm
- net D3.3V: track 0.00 -> 6.68 mm
- net N-00000156: track 0.00 -> 4.44 mm
- net SCL: track 0.00 -> 2.46 mm
- net SDA: track 0.00 -> 2.19 mm
- added copper zone on F.Cu, net /Mosfet Outputs/Bed_Fused
- added copper zone on F.Cu, net /Mosfet Outputs/Ext_Fused
- added copper zone on B.Cu, net ADC_GND
- added copper zone on F.Cu, net ADC_GND
- added copper zone on B.Cu, net DGND
- added copper zone on F.Cu, net DGND
Other:
- board outline added: 99.1 x 99.1 mm
- copper layers 0 -> 2
- net class Default added: clearance 0.2032, trace_width 0.2032, via_dia 0.635, via_drill 0.3048
- net class high-power added: clearance 0.2032, trace_width 2.286, via_dia 2.286, via_drill 1.016
- net class low-power added: clearance 0.2032, trace_width 0.4064, via_dia 0.635, via_drill 0.3048
- net class med-power added: clearance 0.2032, trace_width 1.143, via_dia 1.143, via_drill 0.508
- net class motor-power added: clearance 0.2032, trace_width 1.6002, via_dia 1.6256, via_drill 1.016
- net class power added: clearance 0.2032, trace_width 0.762, via_dia 0.762, via_drill 0.381
- board text added: "0"
- board text added: "1"
- board text added: "2"
- board text added: "3"
- board text added: "A0"
- board text added: "BB ON"
- board text added: "CRAMPS v2.2"
- board text added: "ESTOP"
- board text added: "LIMIT SW"
- board text added: "P8"
- board text added: "P9"
- board text added: "RST"
- board text added: "S"
- board text added: "SERIAL0"
- board text added: "THERM"
- board text added: "WP"
- board text added: "X"
- board text added: "Y"
- board text added: "Z"
- board text added: "reprap.org/wiki/CRAMPS"
- board text added: "© 2014 GPL v3"
