File: RosettaBone_Redux/RBR.sch (KiCad schematic (older format))
At the start: 17 parts, among them M101 PCB_GREEN_RMC, M102 LOGO_OSHW, P101 SOCKET_6_LONG, P102 HEADER_2, P103 HEADER_2, P106 CONN_3X2, P8 BB_EXP_CONN, P9 BB_EXP_CONN, Q101 2N7002K, SW101 SW_PUSH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

Commit message: Cleanup
Parts:
- removed LD101: Yellow, OSRAM-LED-0603, symbol LED
- removed LD102: Green, OSRAM-LED-0603, symbol LED
- removed P102, P103: HEADER_2, pin_strip_2, symbol HEADER_2
- removed P106: CONN_3X2, symbol CONN_3X2
- removed Q101: 2N7002K, SOT23GDS, symbol FET_N
- removed R101, R102: 330R, RESC1608x55N, symbol R
- removed SW101, SW102: SW_PUSH, SW_6x6_MULTI, symbol SW_PUSH
Connections:
- net A4 is gone; now on net AIN0: SHIELD101.AD4
- net A5 is gone; now on net AIN1: SHIELD101.AD5
- net A6 is gone; now on net AIN2: SHIELD101.AD6
- net A7 is gone; now on net AIN3: SHIELD101.AD7
- net D10 is gone; now on net FET3: SHIELD101.10 (D10)
- net D11-FET4 is gone; now on net FET4: SHIELD101.11 (D11)
- net D12-FET5 is gone; now on net FET5: SHIELD101.12 (D12)
- net D13 is gone; now on net FET6: SHIELD101.13 (D13)
- net D39 is gone; now on net AXIS_ENAn: SHIELD101.39 (D39)
- net D45 is gone; now on net AXIS_ENAn: SHIELD101.45 (D45)
- net D8 is gone; now on net FET1: SHIELD101.8 (D8)
- net D9 is gone; now on net FET2: SHIELD101.9 (D9)
- net DUE_5V is gone; now on net +5V: SHIELD101.5V
- net E0_EN is gone; now on net AXIS_ENAn: SHIELD101.42 (D42)
- net LED is gone; now on net FET6: P9.25 (GPIO3_21)
- net RESET is gone; now on net RESETn: SHIELD101.RST
- net THERM3 is gone; now on net AIN0: SHIELD101.AD3
- net X_EN is gone; now on net AXIS_ENAn: SHIELD101.48 (D48)
- net Y_EN is gone; now on net AXIS_ENAn: SHIELD101.46 (D46)
- net Z_EN is gone; now on net AXIS_ENAn: SHIELD101.44 (D44)
- net +3.3V: now also SHIELD101.IORF (IOREF)
- net IOREF: no longer SHIELD101.IORF (IOREF)
- net AD14: no longer names the net of SHIELD101.AD14 (AD14-CANRX)
- net AD15: no longer names the net of SHIELD101.AD15 (AD15-CANTX)
- net AM-VIN: no longer names the net of SHIELD101.V_IN
- net D23: no longer names the net of SHIELD101.23 (D23)
- net D25: no longer names the net of SHIELD101.25 (D25)
- net D27: no longer names the net of SHIELD101.27 (D27)
- net D29: no longer names the net of SHIELD101.29 (D29)
- net D31: no longer names the net of SHIELD101.31 (D31)
- net D33: no longer names the net of SHIELD101.33 (D33)
- net D35: no longer names the net of SHIELD101.35 (D35)
- net D37: no longer names the net of SHIELD101.37 (D37)
- net D49: no longer names the net of SHIELD101.49 (D49)
- net MACHINE_PWR: no longer names the net of P9.23 (GPIO1_17)
- net PWR_BUT: no longer names the net of P9.9 (PWR_BUT)
- net SERVO1: no longer names the net of SHIELD101.7 (D7)
- net SERVO2: no longer names the net of SHIELD101.6 (D6)
- net SERVO3: no longer names the net of SHIELD101.5 (D5)
- net SERVO4: no longer names the net of SHIELD101.3 (D3)
- net UART1_RX_LV: no longer names the net of SHIELD101.19 (D19-RX1)
- net UART1_TX_LV: no longer names the net of SHIELD101.18 (D18-TX1)
- net UART2_RX_LV: no longer names the net of SHIELD101.17 (D17-RX2)
- net UART2_TX_LV: no longer names the net of SHIELD101.16 (D16-TX2)
- net UART3_RX_LV: no longer names the net of SHIELD101.15 (D15-RX3)
- net UART3_TX_LV: no longer names the net of SHIELD101.14 (D14-TX3)
- no-connect marks 39 -> 62
Other:
- note removed: "BB ON\nLED\n"
- note removed: "Power"
- note removed: "Reset"
- note removed: "STATUS\nLED"
- note removed: "To save money on all the pin headers\nwhen buying parts for a few boards,\nyou can get large breakaway headers\ninstead of the individual parts. You\nwill need a total of:\n\n18 pins of single-row header\n82 pins of dual-row header\n\nWhich you can get using\n(1) Harwin M20-9993645 36-pin single-row header\n(2) Harwin M20-9983645 72-pin dual-row header\n\nIf you want to use standard pin headers i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"
- moved on the sheet: P101
