File: RosettaBone_Redux/con_inputs.sch (KiCad schematic (older format))
At the start: 34 parts, among them P501 HEADER_6, P502 HEADER_6X2, P503 HEADER_4X2, P504 HEADER_4X2, U501 74CBTD3861

Commit message: Cleanup
Parts:
- removed C502, C503, C504, C505: 100n, CAPC1608x55N, symbol C
- removed C506, C507, C508, C509: 10u, CAPC1608x55N, symbol C
- removed JP501: HEADER_2, pin_strip_2, symbol JUMP_MINI
- removed P501: HEADER_6, pin_strip_6, symbol HEADER_6
- removed P502: HEADER_6X2, pin_strip_6x2, symbol HEADER_6X2
- removed P503, P504: HEADER_4X2, pin_strip_4x2, symbol HEADER_4X2
- removed R511, R512, R513, R514: 2K0 1%, RESC1608x55N, symbol R
- removed R515, R516, R517, R518: 4k7, RESC1608x55N, symbol R
- removed S501: SHUNT, Shunt, symbol SHUNT
Connections:
- net labels removed: ADC_GND, ADC_VDD, AIN3, THERM0, THERM1, THERM2, THERM3
- wire segments 98 -> 45
Other:
- note removed: "DIR_V"
- note removed: "DIR_W"
- note removed: "From \nThermistors"
- note removed: "P503 may be used for:\n* Additional digital I/O\n* CRAMP3 add-on board\n* SPI expansion"
- note removed: "STEP_V"
- note removed: "STEP_W"
- note removed: "Shunt populated by default\nRemove to support\n4-wire touch-screen\nusing AIN 0-3"
- note removed: "To ADC\nInputs"
