File: RosettaBone_Redux/e-stop.sch (KiCad schematic (older format))
At the start: 34 parts, among them P301 HEADER_2, P302 KK-2.54-2W, P303 HEADER_4X2, P304 HEADER_3X2, P305 HEADER_6, Q301 2N7002K, Q302 2N7002K, Q303 2N7002K, Q304 2N7002K, Q305 2N7002K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

Commit message: Cleanup
Parts:
- removed LD301: Green, OSRAM-LED-0603, symbol LED
- removed LD302: Red, OSRAM-LED-0603, symbol LED
- removed P301: HEADER_2, pin_strip_2, symbol HEADER_2
- removed P302: KK-2.54-2W, CONN_KK_2.54_2W, symbol HEADER_2
- removed P303: HEADER_4X2, pin_strip_4x2, symbol HEADER_4X2
- removed P304: HEADER_3X2, pin_strip_3x2, symbol HEADER_3X2
- removed P305: HEADER_6, pin_strip_6, symbol HEADER_6
- removed Q301, Q302, Q303, Q304, Q305: 2N7002K, SOT23GDS, symbol FET_N
- removed R301: 10k, RESC1608x55N, symbol R
- removed R302: 2K7, RESC1608x55N, symbol R
- removed R303: 330R, RESC1608x55N, symbol R
- removed R304: 4k7, RESC1608x55N, symbol R
- removed R305: 220R, RESC1608x55N, symbol R
- removed S301: SHUNT, Shunt, symbol SHUNT
Connections:
- net labels removed: +V_MOTOR, ADC_GND, ADC_VDD, AIN0, AIN1, AIN2, AIN3, ESTOP, ESTOP_SW, MACHINE_PWR, MACHINE_PWRn, PS-On, SPI_CS1, SPI_SPARE
- wire segments 129 -> 69
Other:
- note removed: "ACTIVE"
- note removed: "ATX Power On"
- note removed: "Analog"
- note removed: "CRAMP3 Expansion"
- note removed: "DIR_U"
- note removed: "ESTOP"
- note removed: "ESTOP Active (high) unless:\n* ESTOP chain is unbroken\n* Software is driving ESTOP_SW low"
- note removed: "Emergency Stop switch\n(Normally Closed type)\nuse shunt if not present"
- note removed: "I2C and misc signals"
- note removed: "Machine Power\nStatus LED"
- note removed: "Motor Power"
- note removed: "Must use ACT type buffer\nwith 24 mA output drive\nInputs are compatible with \n3.3V or 5V logic"
- note removed: "Place a shunt on ESTOP header\nby default, for folks who do not\nhave an off-board ESTOP switch"
- note removed: "Resistive Touch Screen"
- note removed: "STEP_U"
- note removed: "Series resistor on ESTOPn provides\nsome protection from ESTOP chain\n\nFETs protect against high voltage\nfrom PS_ON or MACHINE_PWRn\nfeeding back to the 3.3V 'Bone\n"
- note removed: "Status LED"
- note removed: "Two FETs used to keep ESTOP\npolarity consistent with V1.0"
- note removed: "X+"
- note removed: "X-"
- note removed: "Y+"
- note removed: "Y-"
